Commit message: differential drive controller and head hokuyo laser added to Robot

File: my_rb1_description/urdf/my_rb1_robot.urdf (robot description, URDF)
Before this commit: robot RB1 robot, 7 links, 6 joints
Links:
- removed link link_laser_scan
- added link front_laser, mass 0.25; collision cylinder length=0.20 radius=0.15; visual cylinder length=0.025 radius=0.0125
Joints:
- removed joint joint_chassis_back_caster_wheel
- removed joint joint_chassis_caster_wheel
- removed joint joint_cylinder_left_wheel
- removed joint joint_cylinder_right_wheel
- removed joint joint_laser_scan_chassis
- added joint joint_base_link_back_caster_wheel: type fixed, parent base_link, child back_caster, origin xyz=.1 0 -0.15 rpy=0 0 0
- added joint joint_base_link_front_caster_wheel: type fixed, parent base_link, child front_caster, origin xyz=-.1 0 -0.15 rpy=0 0 0
- added joint joint_base_link_front_laser_: type fixed, parent base_link, child front_laser, origin xyz=0.25 0 0.075 rpy=3.14159 0 0
- added joint joint_base_link_left_wheel: type continuous, parent base_link, child left_wheel, origin xyz=0 .2 -.15 rpy=0 0 0, axis 0 1 0, limit effort=10000 velocity=1000
- added joint joint_base_link_right_wheel: type continuous, parent base_link, child right_wheel, origin xyz=0 -.2 -.15 rpy=0 0 0, axis 0 1 0, limit effort=10000 velocity=1000
